File: sequenception_hw/sequenception_hw/button_matrix.sch (KiCad schematic (older format))
At the start: 128 parts, among them SW17 SW_Push, SW18 SW_Push, SW19 SW_Push, SW20 SW_Push, SW21 SW_Push, SW22 SW_Push, SW23 SW_Push, SW24 SW_Push, SW25 SW_Push, SW26 SW_Push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

Commit message: cleanup repo
Parts:
- renumbered SW18 to SW10, SW19 to SW11, SW20 to SW12, SW21 to SW13, SW22 to SW14, SW23 to SW15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
