File: sequenception_hw/sequenception_hw/sequenception_hw.kicad_pcb (KiCad board)
At the start: 2 copper layers, 124.5 x 194.3 mm, 175 parts, among them J1 MIDI_IN, J2 Conn_01x09_Female, J3 Conn_01x08_Male, J4 Conn_02x08_Odd_Even, J5 MIDI_OUT, J6 SOFTPOT_CONN, J7 Conn_01x02_Male, J8 Conn_01x08_Male, J9 Conn_01x03_Male, SW1 SW_Push, SW10 SW_Push, SW11 SW_Push, SW12 SW_Push, SW17 SW_Push, SW18 SW_Push, SW19 SW_Push, SW2 SW_Push, SW20 SW_Push, SW21 SW_Push, SW22 SW_Push, SW23 SW_Push, SW24 SW_Push, SW25 SW_Push, SW26 SW_Push, SW27 SW_Push, SW28 SW_Push, SW29 SW_Push, SW3 SW_Push, SW30 SW_Push, SW31 SW_Push, SW32 SW_Push, SW33 SW_Push, SW34 SW_Push, SW35 SW_Push, SW36 SW_Push, SW37 SW_Push, SW38 SW_Push, SW39 SW_Push, SW4 SW_Push, SW40 SW_Push, SW41 SW_Push, SW42 SW_Push, SW43 SW_Push, SW44 SW_Push, SW45 SW_Push, SW46 SW_Push, SW47 SW_Push, SW48 SW_Push, SW49 SW_Push, SW50 SW_Push, SW51 SW_Push, SW52 SW_Push, SW53 SW_Push, SW54 SW_Push, SW55 SW_Push, SW56 SW_Push, SW57 SW_Push, SW58 SW_Push, SW59 SW_Push, SW60 SW_Push, SW61 SW_Push, SW62 SW_Push, SW63 SW_Push, SW64 SW_Push, SW65 SW_Push, SW66 SW_Push, SW67 SW_Push, SW68 SW_Push, SW69 SW_Push, SW70 SW_Push, SW71 SW_Push, SW72 SW_Push, SW73 SW_Push, SW74 SW_Push, SW75 SW_Push, SW76 SW_Push, SW77 SW_Push, SW78 SW_Push, SW79 SW_Push, SW80 SW_Push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

Commit message: cleanup repo
Parts:
- removed the J7 at (172.7, 128.3)
- removed REF** (x10): MountingHole_3.2mm_M3, MountingHole:MountingHole_3.2mm_M3
- removed the SW11 at (168.9, 95.2)
- added C4: 0.1uF, Capacitor_THT:C_Disc_D5.0mm_W2.5mm_P2.50mm, B.Cu at (141.0, 100.3)
- added C5: 0.1uF, Capacitor_THT:C_Disc_D5.0mm_W2.5mm_P2.50mm, B.Cu at (109.2, 114.3)
- added C6: 0.1uF, Capacitor_THT:C_Disc_D5.0mm_W2.5mm_P2.50mm, B.Cu at (116.8, 105.4)
- added H1: MountingHole, MountingHole:MountingHole_3.2mm_M3, F.Cu at (143.5, 81.3)
- added H10: MountingHole, MountingHole:MountingHole_3.2mm_M3, F.Cu at (55.9, 246.4)
- added H2: MountingHole, MountingHole:MountingHole_3.2mm_M3, F.Cu at (81.3, 116.8)
- added H3: MountingHole, MountingHole:MountingHole_3.2mm_M3, F.Cu at (170.2, 62.2)
- added H4: MountingHole, MountingHole:MountingHole_3.2mm_M3, F.Cu at (81.3, 81.3)
- added H5: MountingHole, MountingHole:MountingHole_3.2mm_M3, F.Cu at (55.9, 62.2)
- added H6: MountingHole, MountingHole:MountingHole_3.2mm_M3, F.Cu at (143.5, 116.8)
- added H7: MountingHole, MountingHole:MountingHole_3.2mm_M3, F.Cu at (170.2, 158.8)
- added H8: MountingHole, MountingHole:MountingHole_3.2mm_M3, F.Cu at (55.9, 158.8)
- added H9: MountingHole, MountingHole:MountingHole_3.2mm_M3, F.Cu at (170.2, 246.4)
- added SW6: SW_Push, Button_Switch_THT:SW_PUSH_6mm, F.Cu at (157.5, 105.4)
- C2: renamed from C3; footprint Capacitor_THT:C_Radial_D5.0mm_H5.0mm_P2.00mm -> Capacitor_THT:C_Disc_D5.0mm_W2.5mm_P2.50mm
- C3: renamed from C2; footprint Capacitor_THT:C_Radial_D5.0mm_H5.0mm_P2.00mm -> Capacitor_THT:C_Disc_D5.0mm_W2.5mm_P2.50mm
- moved SW7 15.3 mm to (168.9, 105.4)
- moved J5 12.8 mm to (171.4, 130.8)
- moved SW5 10.2 mm to (168.9, 95.2)
- moved SW8 10.2 mm to (157.5, 95.2)
- moved D2 9.25 mm to (168.9, 115.6), turned to 90 degrees
- moved R6 7.73 mm to (163.8, 110.5), turned to 180 degrees
- moved R8 7.73 mm to (163.8, 118.1), turned to 180 degrees
- moved R7 1.27 mm to (163.8, 114.3), turned to 180 degrees
- renumbered J3 to J1, J1 to J2, J2 to J3, J9 to J5, J5 to J6, J6 to J7, SW18 to SW10, SW19 to SW11, SW20 to SW12, SW21 to SW13, SW22 to SW14, SW23 to SW15, SW24 to SW16, SW25 to SW17, SW26 to SW18, SW27 to SW19, SW28 to SW20, SW29 to SW21, SW30 to SW22, SW31 to SW23, SW32 to SW24, SW33 to SW25, SW34 to SW26, SW35 to SW27, SW36 to SW28, SW37 to SW29, SW38 to SW30, SW39 to SW31, SW40 to SW32, SW41 to SW33, SW42 to SW34, SW43 to SW35, SW44 to SW36, SW45 to SW37, SW46 to SW38, SW47 to SW39, SW48 to SW40, SW49 to SW41, SW50 to SW42, SW51 to SW43, SW52 to SW44, SW53 to SW45, SW54 to SW46, SW55 to SW47, SW56 to SW48, SW57 to SW49, SW9 to SW5, SW58 to SW50, SW59 to SW51, SW60 to SW52, SW61 to SW53, SW62 to SW54, SW63 to SW55, SW64 to SW56, SW65 to SW57, SW66 to SW58, SW67 to SW59, SW68 to SW60, SW69 to SW61, SW70 to SW62, SW71 to SW63, SW72 to SW64, SW73 to SW65, SW74 to SW66, SW75 to SW67, SW76 to SW68, SW77 to SW69, SW10 to SW7, SW78 to SW70, SW79 to SW71, SW80 to SW72, SW12 to SW8, SW17 to SW9
Connections:
- J8 pad 5: /GPB4 -> /GPA3
- J8 pad 6: /GPB5 -> /GPA2
- J8 pad 7: /GPB6 -> /GPA1
- J8 pad 8: /GPB7 -> /GPA0
- SW5 pad 1: Net-(SW9-Pad1) -> Net-(SW5-Pad1)
- SW7 pad 1: Net-(SW10-Pad1) -> Net-(SW7-Pad1)
- SW8 pad 1: Net-(SW12-Pad1) -> Net-(SW8-Pad1)
- U2 pad 32: /PIN_AGND -> (no net)
- U2 pad 35: /PIN_AREF -> (no net)
- U3 pad 21: Net-(SW9-Pad1) -> /GPA0
- U3 pad 22: Net-(SW10-Pad1) -> /GPA1
- U3 pad 23: Net-(SW11-Pad1) -> /GPA2
- U3 pad 24: Net-(SW12-Pad1) -> /GPA3
- U3 pad 5: /GPB4 -> Net-(SW8-Pad1)
- U3 pad 6: /GPB5 -> Net-(SW5-Pad1)
- U3 pad 7: /GPB6 -> Net-(SW6-Pad1)
- U3 pad 8: /GPB7 -> Net-(SW7-Pad1)
Routing:
- net +3V3: track 43.7 -> 186.8 mm, vias 0 -> 1
- net GND: track 128.6 -> 0.00 mm
- net Net-(SW5-Pad1): track 0.00 -> 115.3 mm
- net Net-(SW6-Pad1): track 0.00 -> 108.6 mm
- net Net-(SW7-Pad1): track 0.00 -> 107.8 mm
- net Net-(SW8-Pad1): track 0.00 -> 100.0 mm, vias 0 -> 1
- net /SP: track 15.9 -> 92.5 mm, vias 0 -> 3
- net +5V: track 14.6 -> 77.8 mm
- net /PIN12: track 0.00 -> 52.8 mm, vias 0 -> 1
- net /RED: track 0.00 -> 44.7 mm
- net /PIN10: track 0.00 -> 44.3 mm
- net /BLUE: track 0.00 -> 44.2 mm
- net /GPA0: track 0.00 -> 42.0 mm
- net /GPA1: track 0.00 -> 38.4 mm
- net /GPB7: track 37.8 -> 0.00 mm
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- added copper zone on B.Cu, net GND
- added copper zone on F.Cu, net GND
Other:
- net class Power added: clearance 0.25, trace_width 0.38, via_dia 0.8, via_drill 0.4
- board text added: "Sequenception proto 1 Pour ma merveilleuse Aëlle"
