File: sequenception_hw/sequenception_hw/sequenception_hw.sch (KiCad schematic (older format))
At the start: 37 parts, among them J1 MIDI_IN, J2 Conn_01x09_Female, J3 Conn_01x08_Male, J4 Conn_02x08_Odd_Even, J5 MIDI_OUT, J6 SOFTPOT_CONN, J7 Conn_01x02_Male, J8 Conn_01x08_Male, J9 Conn_01x03_Male, SW1 SW_Push, SW10 SW_Push, SW11 SW_Push, SW12 SW_Push, SW2 SW_Push, SW3 SW_Push, SW4 SW_Push, SW9 SW_Push, U1 6N138, U2 Teensy3.2-teensy, U3 MCP23017_SP

Commit message: cleanup repo
Parts:
- removed J7: Conn_01x02_Male, Connector_PinHeader_2.54mm:PinHeader_1x02_P2.54mm_Vertical, symbol Connector:Conn_01x02_Male
- added C4, C5, C6: 0.1uF, Capacitor_THT:C_Disc_D5.0mm_W2.5mm_P2.50mm, symbol Device:C
- added H1, H10, H2, H3, H4, H5, H6, H7, H8, H9: MountingHole, MountingHole:MountingHole_3.2mm_M3, symbol Mechanical:MountingHole
- C2: renamed from C3; footprint Capacitor_THT:C_Radial_D5.0mm_H5.0mm_P2.00mm -> Capacitor_THT:C_Disc_D5.0mm_W2.5mm_P2.50mm
- C3: renamed from C2; footprint Capacitor_THT:C_Radial_D5.0mm_H5.0mm_P2.00mm -> Capacitor_THT:C_Disc_D5.0mm_W2.5mm_P2.50mm
- renumbered J3 to J1, J1 to J2, J2 to J3, J9 to J5, J5 to J6, J6 to J7, SW9 to SW5, SW11 to SW6, SW10 to SW7, SW12 to SW8
Connections:
- net labels added: GPA0, GPA1, GPA2, GPA3
- net labels removed: GPB4, GPB5, GPB6, GPB7, PIN_AGND, PIN_AREF
- wire segments 125 -> 123
- no-connect marks 20 -> 24
Other:
- moved on the sheet: C3, SW5, SW6, SW7, SW8
